File: Adafruit 1.54inch 240x240.sch (EAGLE design)
At the start: 21 parts, among them IC1 4050D, IC2 AP2112, Q2 MICROSD, Q3 BSS138

Commit message: Updating board files.
Parts:
- removed DISP1: DISP_LCD_ST7789_1.54IN, microbuilder:DISP_LCD_ST7789_1.54IN
- removed IC1: 4050D, 40xx:4050D
- removed JP1: (no value), microbuilder:HEADER-1X1176MIL
- removed U$3: FIDUCIAL_1MM, microbuilder:FIDUCIAL_1MM
- added C3, C5: 0.1uF, microbuilder:CAP_CERAMIC0603_NO
- added IC4: APX803-SAG, adafruit:AXP083-SAG
- added JP2: (no value), microbuilder:HEADER-1X1276MIL
- added TFT1: DISP_TFT_1.54IN_240X240_22P, microbuilder:DISP_TFT_1.54IN_240X240_22P
- added U1: 74HC4050PWR, microbuilder:74HC4050DTSSOP
- C4: value 0.1uF -> 10uF
- R1, R2, R4, R5: device microbuilder:RESISTOR0805_NOOUTLINE -> microbuilder:RESISTOR_0603_NOOUT
- R3: value 2.2K -> 10K; device microbuilder:RESISTOR0805_NOOUTLINE -> microbuilder:RESISTOR_0603_NOOUT
Connections:
- new net TE: JP2.12, TFT1.TE
- net +3V3: now also C3.1, C5.1, JP2.2, TFT1.IM1, TFT1.IM2, TFT1.LEDA, TFT1.VCI, U1.VCC; no longer DISP1.LEDA, DISP1.VCC, IC1P.VDD, JP1.2
- net CARDCS: now also JP2.10, U1.4A; no longer IC1F.I, JP1.10
- net CARDCS_3V: now also U1.4Y; no longer IC1F.O
- net GND: now also C3.2, C5.2, IC4.GND, JP2.3, TFT1.!RD, TFT1.DB0, TFT1.DB1, TFT1.DB2, TFT1.DB3, TFT1.DB4, TFT1.DB5, TFT1.DB6, TFT1.DB7, TFT1.GND, TFT1.IM0, U1.GND; no longer DISP1.GND, DISP1.MT1, DISP1.MT2, IC1P.VSS, JP1.3
- net LEDK: now also TFT1.LEDK; no longer DISP1.LEDK
- net LITE: now also JP2.11; no longer JP1.11
- net MISO: now also JP2.5; no longer JP1.5
- net MOSI: now also JP2.6, U1.5A; no longer IC1B.I, JP1.6
- net MOSI_3V: now also TFT1.SDA, U1.5Y; no longer DISP1.DATA, IC1B.O
- net SCK: now also JP2.4, U1.2A; no longer IC1A.I, JP1.4
- net SCK_3V: now also TFT1.RS/CLK, U1.2Y; no longer DISP1.CLOCK, IC1A.O
- net TFTCS: now also JP2.7, U1.1A; no longer IC1C.I, JP1.7
- net TFTCS_3V: now also TFT1.!CS, U1.1Y; no longer DISP1.CS, IC1C.O
- net TFTDC: now also JP2.9, U1.3A; no longer IC1E.I, JP1.9
- net TFTDC_3V: now also TFT1.!WR!/D!C, U1.3Y; no longer DISP1.RS/DC, IC1E.O
- net TFTRST: now also IC4./RESET, JP2.8, U1.6A; no longer IC1D.I, JP1.8
- net TFTRST_3V: now also TFT1.RESET, U1.6Y; no longer DISP1.RST, IC1D.O
- net VIN: now also IC4.VCC, JP2.1; no longer JP1.1
Other:
- moved on the sheet: C1, C2, C4, IC2, R1
